Commit message: Add Imu

File: my_robot_description/urdf/imu.xacro (robot description, xacro)
@@ -25,3 +25,16 @@
         <origin xyz="${2* imu_width} 0 ${base_height}" rpy="0 ${pi/2} 0" />
     </joint>
+    <gazebo reference="imu_link">
+        <material>Gazebo/Red</material>
+        <sensor name="my_imu" type="imu">
+            <always_on>true</always_on>
+            <update_rate>100</update_rate>
+            <plugin name="imu_link" filename="libgazebo_ros_imu_sensor.so">
+                <ros>
+                  <!-- <namespace>/tb3</namespace> -->
+                  <remapping>~/out:=imu</remapping>
+                </ros>
+              </plugin>
+          </sensor>
+      </gazebo>
 </robot>
